File: PCB/BREAD_Slice_V2/BREAD_slice_v2/BREAD_slice_v2.kicad_sch (KiCad schematic)
At the start: 36 parts, among them J1 10018783-10200TLF, J10 Screw_Terminal_01x04, J11 Screw_Terminal_01x04, J2 Screw_Terminal_01x04, J3 Conn_01x03_Male, J4 Conn_01x06_Socket, J5 Screw_Terminal_01x02, J6 Conn_01x02_Socket, J7 Conn_01x10_Socket, J8 Screw_Terminal_01x04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

Commit message: fixed can tx/rx on input only pins
Connections:
- net AG_1: now also U1.J2_3 (SENSOR_VP); no longer U1.J2_7 (IO32)
- net AG_2: now also U1.J2_4 (SENSOR_VN); no longer U1.J2_8 (IO33)
- net AG_3: now also U1.J2_5 (IO34); no longer U1.J2_9 (IO25)
- net AG_4: now also U1.J2_6 (IO35); no longer U1.J2_10 (IO26)
- net EstpCh1: now also U1.J2_7 (IO32); no longer U1.J2_3 (SENSOR_VP)
- net EstpCh2: now also U1.J2_8 (IO33); no longer U1.J2_4 (SENSOR_VN)
- net RX: now also U1.J2_10 (IO26); no longer U1.J2_6 (IO35)
- net TX: now also U1.J2_9 (IO25); no longer U1.J2_5 (IO34)
Changed lines of the file:
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@@
-		)
-	)
-	(label "AG_4"
-		(at 24.13 81.28 0)
-		(effects
-			(font
-				(size 1.27 1.27)
-			)
-			(justify left bottom)
 		)
 	)
@@
 		)
 	)
-	(label "TX"
-		(at 24.13 68.58 0)
-		(effects
-			(font
-				(size 1.27 1.27)
-			)
-			(justify left bottom)
-		)
-	)
 	(label "DR_3"
 		(at 80.01 88.9 180)
@@
 		)
 	)
-	(label "AG_2"
-		(at 24.13 76.2 0)
-		(effects
-			(font
-				(size 1.27 1.27)
-			)
-			(justify left bottom)
-		)
-	)
 	(label "SYNC"
 		(at 24.13 93.98 0)
@@
 		)
 	)
+	(label "AG_3"
+		(at 24.13 68.58 0)
+		(effects
+			(font
+				(size 1.27 1.27)
+			)
+			(justify left bottom)
+		)
+	)
 	(label "A3_1B"
 		(at 229.87 54.61 180)
@@
 		)
 	)
-	(label "RX"
-		(at 24.13 71.12 0)
-		(effects
-			(font
-				(size 1.27 1.27)
-			)
-			(justify left bottom)
-		)
-	)
 	(label "A_IN4"
 		(at 153.67 109.22 0)
@@
 		)
 	)
+	(label "RX"
+		(at 24.13 81.28 0)
+		(effects
+			(font
+				(size 1.27 1.27)
+			)
+			(justify left bottom)
+		)
+	)
 	(label "ST_3"
 		(at 80.01 86.36 180)
@@
 		)
 	)
-	(label "AG_3"
-		(at 24.13 78.74 0)
-		(effects
-			(font
-				(size 1.27 1.27)
-			)
-			(justify left bottom)
-		)
-	)
 	(label "EstpCh1"
 		(at 35.56 165.1 0)
@@
 		)
 	)
+	(label "AG_4"
+		(at 24.13 71.12 0)
+		(effects
+			(font
+				(size 1.27 1.27)
+			)
+			(justify left bottom)
+		)
+	)
 	(label "SDA"
 		(at 223.52 116.84 0)
@@
 		)
 	)
+	(label "EstpCh2"
+		(at 24.13 76.2 0)
+		(effects
+			(font
+				(size 1.27 1.27)
+			)
+			(justify left bottom)
+		)
+	)
 	(label "A4_1B"
 		(at 259.08 125.73 0)
@@
 		)
 	)
+	(label "EstpCh1"
+		(at 24.13 73.66 0)
+		(effects
+			(font
+				(size 1.27 1.27)
+			)
+			(justify left bottom)
+		)
+	)
 	(label "ST_3"
 		(at 193.04 57.15 0)
@@
 		)
 	)
-	(label "AG_1"
-		(at 24.13 73.66 0)
-		(effects
-			(font
-				(size 1.27 1.27)
-			)
-			(justify left bottom)
-		)
-	)
 	(label "DR_4"
 		(at 80.01 93.98 180)
@@
 		)
 	)
+	(label "AG_1"
+		(at 24.13 63.5 0)
+		(effects
+			(font
+				(size 1.27 1.27)
+			)
+			(justify left bottom)
+		)
+	)
 	(label "DR_1"
 		(at 107.95 59.69 0)
@@
 		)
 	)
+	(label "TX"
+		(at 24.13 78.74 0)
+		(effects
+			(font
+				(size 1.27 1.27)
+			)
+			(justify left bottom)
+		)
+	)
 	(label "ST_4"
 		(at 237.49 57.15 0)
@@
 		)
 	)
+	(label "AG_2"
+		(at 24.13 66.04 0)
+		(effects
+			(font
+				(size 1.27 1.27)
+			)
+			(justify left bottom)
+		)
+	)
 	(label "MS3"
 		(at 149.86 64.77 0)
@@
 		)
 	)
-	(label "EstpCh1"
-		(at 24.13 63.5 0)
-		(effects
-			(font
-				(size 1.27 1.27)
-			)
-			(justify left bottom)
-		)
-	)
 	(label "M_POWER"
 		(at 201.93 115.57 180)
@@
 		(effects
 			(font
-				(size 1.27 1.27)
-			)
-			(justify left bottom)
-		)
-	)
-	(label "EstpCh2"
-		(at 24.13 66.04 0)
-		(effects
-			(font
